File: controller/controller.kicad_pcb (KiCad board)
At the start: 2 copper layers, 130 x 60 mm, 34 parts, among them J1 Arduino_Nano_Header, P1 CONN_01X03, P2 CONN_01X03, P3 CONN_01X07, P4 CONN_01X02, SW1 DIPS_10, U1 MAX5024, U3 IL610, U4 MAX3040, U5 74LS165, U6 74LS165

Commit message: REV1 boards ordered
Parts:
- added P5: CONN_01X11, Pin_Headers:Pin_Header_Straight_1x11, F.Cu at (139.2, 100.8)
- added P6: CONN_01X08, Pin_Headers:Pin_Header_Straight_1x08, F.Cu at (139.1, 77.3)
- added REF**: MountingHole_3.2mm_M3, Mounting_Holes:MountingHole_3.2mm_M3, F.Cu at (90.0, 109.0)
- added REF**: MountingHole_3.2mm_M3, Mounting_Holes:MountingHole_3.2mm_M3, F.Cu at (90.0, 88.0)
- moved TH1 22.5 mm to (118.1, 75.8)
- moved C8 15.0 mm to (99.7, 89.7)
- moved C9 15.0 mm to (105.0, 83.0), turned to 90 degrees
- moved P3 15.0 mm to (97.0, 91.3)
- moved C6 8.30 mm to (113.1, 94.2), turned to 90 degrees
- moved U4 8.00 mm to (107.0, 98.0)
- moved C7 1.90 mm to (138.1, 84.9), turned to 180 degrees
Connections:
- J1 pad 27: +5V -> Net-(J1-Pad27)
- J1 pad 28: Net-(J1-Pad28) -> /RESET
- J1 pad 30: Net-(J1-Pad30) -> +5V
- U1 pad 4: Net-(U1-Pad4) -> /RESET
- U1 pad 9: (no net) -> GND
Routing:
- net /RESET: track 0.00 -> 66.9 mm, vias 0 -> 2
- net VCC: track 124.4 -> 101.5 mm
- net GND: track 92.6 -> 113.9 mm, vias 22 -> 40
- net +5V: track 262.6 -> 247.7 mm, vias 5 -> 3
- net Net-(J1-Pad7): track 61.8 -> 50.9 mm
- net Net-(P3-Pad5): track 19.8 -> 12.2 mm
- net Net-(P3-Pad2): track 23.8 -> 16.6 mm
- net Net-(P3-Pad3): track 21.5 -> 14.3 mm
- net Net-(P3-Pad4): track 16.8 -> 9.95 mm
- net Net-(C8-Pad1): track 36.7 -> 31.6 mm
- net Net-(J1-Pad25): track 0.00 -> 5.09 mm
- net Net-(J1-Pad24): track 0.00 -> 5.09 mm
- net Net-(J1-Pad23): track 0.00 -> 5.09 mm
- net Net-(J1-Pad22): track 0.00 -> 5.09 mm
- net Net-(J1-Pad21): track 0.00 -> 5.09 mm
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Other:
- outline, holes or cut-outs redrawn
