File: controller/controller.kicad_pcb (KiCad board)
At the start: 2 copper layers, 130 x 60 mm, 38 parts, among them J1 Arduino_Nano_Header, P1 CONN_01X03, P2 CONN_01X03, P3 CONN_01X07, P4 CONN_01X02, P5 CONN_01X11, P6 CONN_01X08, SW1 DIPS_10, U1 MAX5024, U3 IL610, U4 MAX3040, U5 74LS165, U6 74LS165

Commit message: Add fixes to PCB
Parts:
- added R4: R, Resistors_SMD:R_0603_HandSoldering, B.Cu at (129.9, 106.1)
- P5: value CONN_01X11 -> CONN_01X10; footprint Pin_Headers:Pin_Header_Straight_1x11 -> Pin_Headers:Pin_Header_Straight_1x10
- moved P5 2.56 mm to (141.8, 100.8)
- moved C5 2.28 mm to (131.0, 103.2), turned to 180 degrees
- moved U3 1.90 mm to (134.6, 106.9)
- moved R1 0.54 mm to (199.7, 107.2)
Connections:
- J1 pad 14: /DATA -> Net-(J1-Pad14)
- J1 pad 15: Net-(J1-Pad15) -> /DATA
- P5 pad 1: Net-(J1-Pad5) -> Net-(J1-Pad6)
- P5 pad 2: Net-(J1-Pad6) -> Net-(J1-Pad7)
- P5 pad 3: Net-(J1-Pad7) -> Net-(J1-Pad8)
- P5 pad 4: Net-(J1-Pad8) -> Net-(J1-Pad9)
- P5 pad 5: Net-(J1-Pad9) -> Net-(J1-Pad10)
- P5 pad 6: Net-(J1-Pad10) -> Net-(J1-Pad11)
- P5 pad 7: Net-(J1-Pad11) -> /DXM_OK
- P5 pad 8: /DXM_OK -> /LATCH
- P5 pad 9: /LATCH -> Net-(J1-Pad14)
- U3 pad 7: GND -> Net-(J1-Pad5)
- U6 pad 10: Net-(RP1-Pad2) -> Net-(U6-Pad10)
- U6 pad 11: Net-(R1-Pad1) -> Net-(RP1-Pad2)
- U6 pad 12: GND -> Net-(R1-Pad1)
Routing:
- net Net-(J1-Pad5): track 3.22 -> 16.2 mm, vias 0 -> 2
- net Net-(J1-Pad14): track 0.00 -> 3.65 mm
- net Net-(J1-Pad15): track 3.22 -> 0.00 mm
- net /DATA: track 29.8 -> 26.9 mm
- net Net-(P1-Pad2): track 62.6 -> 64.9 mm
- net Net-(RP1-Pad2): track 18.3 -> 20.3 mm
- net Net-(R1-Pad1): track 20.6 -> 22.3 mm
- net +5V: track 247.7 -> 249.4 mm
- net Net-(J1-Pad7): track 50.9 -> 52.3 mm
- net Net-(J1-Pad2): track 12.3 -> 13.5 mm
- net Net-(J1-Pad8): track 45.7 -> 46.5 mm
- net Net-(U6-Pad10): track 0.00 -> 0.68 mm
- net Net-(P1-Pad3): track 52.8 -> 52.3 mm
