File: driver/driver.sch (KiCad schematic (older format))
At the start: 11 parts, among them P1 CONN_01X06, P2 CONN_02X03, P3 CONN_01X04, U2 MAX3093, U3 MAX5024

Commit message: REV1 boards ordered
Changed lines of the file:
@@
 	3700 4050 3700 4700
 Wire Wire Line
-	5750 3000 5850 3000
-Wire Wire Line
-	5850 3000 5950 3000
-Wire Wire Line
-	5950 3000 6150 3000
+	5750 3000 6150 3000
 Connection ~ 5950 3000
 Connection ~ 5850 3000
@@
 $EndComp
 Wire Wire Line
-	5100 2150 5250 2150
-Wire Wire Line
-	5250 2150 5600 2150
+	5100 2150 5600 2150
 Connection ~ 3300 2450
 Wire Wire Line
-	3050 2150 3300 2150
-Wire Wire Line
-	3300 2150 3650 2150
-Wire Wire Line
-	3650 2150 3800 2150
+	3050 2150 3800 2150
 $Comp
 L GND #PWR014
