File: driver/driver.kicad_pcb (KiCad board)
At the start: 2 copper layers, 50 x 50 mm, 15 parts, among them P1 CONN_01X06, P2 CONN_02X03, P3 CONN_01X04, U2 MAX3093, U3 MAX5024

Commit message: REV1 boards ordered
Parts:
- moved P1 3.00 mm to (142.0, 61.4)
- moved C6 1.87 mm to (133.7, 69.3), turned to 0 degrees
Connections:
- C6 pad 1: Net-(C6-Pad1) -> VCC
- DRV1 pad 5: +5V -> Net-(DRV1-Pad5)
- P1 pad 1: Net-(C6-Pad1) -> Net-(P1-Pad1)
- TH1 pad 2: Net-(C6-Pad1) -> Net-(P1-Pad1)
- U3 pad 1: Net-(C6-Pad1) -> VCC
- U3 pad 2: Net-(C6-Pad1) -> VCC
- U3 pad 4: Net-(U3-Pad4) -> Net-(DRV1-Pad5)
- U3 pad 9: (no net) -> GND
Routing:
- net Net-(C6-Pad1): track 25.5 -> 0.00 mm
- net Net-(DRV1-Pad5): track 0.00 -> 15.6 mm
- net Net-(P1-Pad1): track 0.00 -> 12.8 mm
- net VCC: track 23.1 -> 33.4 mm
- net GND: track 23.7 -> 30.7 mm, vias 9 -> 14
- net Net-(P1-Pad4): track 11.5 -> 7.88 mm
- net Net-(P1-Pad5): track 9.48 -> 6.48 mm
- net +5V: track 59.6 -> 57.0 mm
- net Net-(P1-Pad3): track 17.8 -> 15.3 mm
- net Net-(P1-Pad2): track 19.9 -> 18.5 mm
Other:
- outline, holes or cut-outs redrawn

Commit message: Clean up even more
Parts:
- DRV1: footprint drv8825:DRV8825 -> fresnel:DRV8825
